File: hardware/PCB/Aero_hand_open_right/Aero-Hand-Open-Right.kicad_sch (KiCad schematic)
At the start: 27 parts, among them J1 22-03-5035, J2 22-03-5035, J3 22-03-5035, J4 22-03-5035, J5 22-03-5035, J6 22-03-5035, J7 22-03-5035, J8 XT30PW-M, Q1 MMBT2907A, U1 SN74LVC1G126DBVR, U2 SN74LVC1G125DBVR, U3 XIAO-ESP32-S3-DIP

Commit message: Rebrand TetherIA → Chestnut Robotics; move links to the chestnut-robotics org
TetherIA, Inc. is now Chestnut Robotics, Inc. (same legal entity, renamed).
- Repository, org, project-page and raw-asset URLs → github.com/chestnut-robotics
- Company site → https://chestnut.bot; mailboxes → the same names @chestnut.bot
- Copyright / NOTICE lines → Chestnut Robotics, Inc. (formerly TetherIA, Inc.);
  per-file headers → Chestnut Robotics, Inc.
- LICENSE.md: name-change note, attribution and trademark wording
- Logo assets (sdk/assets, firmware/main/assets) → Chestnut Robotics wordmark
- Fix Discussions/Issues badges that pointed at RoboVerseOrg/RoboVerse
- SDK metadata GitHub URL now points at the public sdk/ folder (old target is a private repo)

Unchanged on purpose: docs.tetheria.ai links (until the docs domain moves), shop URL,
X/YouTube/LinkedIn handles, MuJoCo Menagerie directory name, RL checkpoint filename.
Other:
- company: TetherIA -> Chestnut Robotics
Changed lines of the file:
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@@
 		(date "2025-09-24")
 		(rev "Rev_V0")
-		(company "TetherIA")
+		(company "Chestnut Robotics")
 	)
 	(junction
